File: abeille/abeille_weight/abeille_weight.kicad_pcb (KiCad board)
At the start: 2 copper layers, 76.2 x 19 mm, 22 parts, among them P1 HE10-10, U1 CD4052B

Commit message: update abeille weight project
Parts:
- added P2: CONN_01X06, Pin_Headers:Pin_Header_Straight_1x06, F.Cu at (245.1, 113.0)
- added P3: CONN_01X04, Pin_Headers:Pin_Header_Straight_1x04, F.Cu at (224.8, 123.2)
- moved RVAR4 10.2 mm to (194.3, 124.5), turned to 270 degrees
- moved RVAR1 8.52 mm to (189.2, 115.6), turned to 90 degrees
- moved RVAR2 1.27 mm to (194.3, 115.6)
- moved RVAR3 1.27 mm to (189.2, 124.5)
Connections:
- P1 pad 6: (no net) -> /SCK
- P1 pad 8: (no net) -> /DT
- U1 pad 16: (no net) -> +5V
Routing:
- net +5V: track 92.6 -> 153.0 mm, vias 3 -> 4
- net GND: track 139.4 -> 180.8 mm
- net /XCOM: track 3.07 -> 43.1 mm, vias 0 -> 1
- net /YCOM: track 23.7 -> 58.1 mm
- net /SCK: track 0.00 -> 21.2 mm
- net /DT: track 0.00 -> 21.2 mm
- net Net-(R9-Pad2): track 30.0 -> 9.42 mm, vias 0 -> 2
- net Net-(R11-Pad1): track 70.8 -> 81.9 mm, vias 3 -> 1
- net Net-(R12-Pad2): track 18.1 -> 13.2 mm
- net Net-(R10-Pad2): track 13.5 -> 14.8 mm
- net Net-(U1-Pad15): track 67.1 -> 68.1 mm
- net Net-(R11-Pad2): track 7.62 -> 8.15 mm
Other:
- board size 76.2 x 19 mm -> 101.6 x 19 mm
- board text added: "HX711"
- board text added: "module"

Commit message: minor modif
Parts:
- moved WEIGHT3 2.54 mm to (152.4, 121.9)
- moved WEIGHT4 2.54 mm to (152.4, 124.5)
Routing:
- net Net-(U1-Pad11): track 54.4 -> 60.5 mm
- net Net-(U1-Pad15): track 68.1 -> 69.2 mm
Changed lines of the file:
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@@
     (area 147.244999 110.414999 248.995001 129.615001)
     (thickness 1.6)
-    (drawings 8)
-    (tracks 227)
+    (drawings 12)
+    (tracks 236)
     (zones 0)
     (modules 24)
@@
     (0 F.Cu signal)
     (31 B.Cu signal)
-    (33 F.Adhes user hide)
-    (35 F.Paste user hide)
+    (33 F.Adhes user)
+    (35 F.Paste user)
     (37 F.SilkS user)
-    (39 F.Mask user hide)
-    (40 Dwgs.User user hide)
-    (41 Cmts.User user hide)
-    (42 Eco1.User user hide)
-    (43 Eco2.User user hide)
-    (44 Edge.Cuts user hide)
-    (45 Margin user hide)
-    (47 F.CrtYd user hide)
-    (49 F.Fab user hide)
+    (39 F.Mask user)
+    (40 Dwgs.User user)
+    (41 Cmts.User user)
+    (42 Eco1.User user)
+    (43 Eco2.User user)
+    (44 Edge.Cuts user)
+    (45 Margin user)
+    (47 F.CrtYd user)
+    (49 F.Fab user)
   )
   (setup
@@
   )
   (module PIN_ARRAY_3X1 (layer F.Cu)
-    (at 152.4 124.46)
+    (at 152.4 121.92)
     (descr "Connecteur 3 pins")
     (tags "CONN DEV")
-    (fp_text reference WEIGHT3 (at 0.254 -2.159) (layer F.SilkS)
+    (fp_text reference WEIGHT3 (at 7.62 2.54 90) (layer F.SilkS)
       (effects (font (size 1.016 1.016) (thickness 0.1524)))
     )
@@
     (descr "Connecteur 3 pins")
     (tags "CONN DEV")
-    (fp_text reference WEIGHT2 (at 0.254 -2.159) (layer F.SilkS)
+    (fp_text reference WEIGHT2 (at 7.62 -1.27 90) (layer F.SilkS)
       (effects (font (size 1.016 1.016) (thickness 0.1524)))
     )
@@
   )
   (module PIN_ARRAY_3X1 (layer F.Cu)
-    (at 152.4 121.92)
+    (at 152.4 124.46)
     (descr "Connecteur 3 pins")
     (tags "CONN DEV")
-    (fp_text reference WEIGHT4 (at 0.254 -2.159) (layer F.SilkS)
+    (fp_text reference WEIGHT4 (at 0 2.54 180) (layer F.SilkS)
       (effects (font (size 1.016 1.016) (thickness 0.1524)))
     )
@@
     )
   )
+  (gr_line (start 157.48 121.92) (end 158.75 123.19) (angle 90) (layer F.SilkS) (width 0.2))
+  (gr_line (start 156.21 121.92) (end 157.48 121.92) (angle 90) (layer F.SilkS) (width 0.2))
+  (gr_line (start 157.48 116.84) (end 158.75 115.57) (angle 90) (layer F.SilkS) (width 0.2))
+  (gr_line (start 156.21 116.84) (end 157.48 116.84) (angle 90) (layer F.SilkS) (width 0.2))
   (gr_text module (at 234.95 121.92) (layer F.SilkS)
     (effects (font (size 1 1) (thickness 0.25)))
@@
   (gr_line (start 147.32 110.49) (end 223.52 110.49) (angle 90) (layer Edge.Cuts) (width 0.15))
   (gr_line (start 147.32 110.49) (end 147.32 129.54) (angle 90) (layer Edge.Cuts) (width 0.15))
+  (segment (start 152.4 124.46) (end 152.4 121.92) (width 0.254) (layer F.Cu) (net 1))
   (segment (start 205.74 123.19) (end 207.01 121.92) (width 0.254) (layer F.Cu) (net 1))
   (segment (start 217.17 118.11) (end 219.71 120.65) (width 0.254) (layer F.Cu) (net 1))
@@
   (segment (start 161.29 123.19) (end 161.29 119.38) (width 0.254) (layer F.Cu) (net 1))
   (segment (start 152.4 119.38) (end 161.29 119.38) (width 0.254) (layer F.Cu) (net 1))
-  (segment (start 152.4 121.92) (end 152.4 124.46) (width 0.254) (layer F.Cu) (net 1))
   (segment (start 152.4 116.84) (end 152.4 119.38) (width 0.254) (layer F.Cu) (net 1))
   (segment (start 152.4 119.38) (end 152.4 121.92) (width 0.254) (layer F.Cu) (net 1))
@@
   (segment (start 220.98 124.46) (end 220.98 121.92) (width 0.254) (layer F.Cu) (net 5))
   (segment (start 214.63 124.46) (end 220.98 124.46) (width 0.254) (layer F.Cu) (net 5))
+  (segment (start 149.86 121.92) (end 149.86 124.46) (width 0.254) (layer F.Cu) (net 6))
   (segment (start 218.44 116.84) (end 227.33 116.84) (width 0.254) (layer B.Cu) (net 6))
   (segment (start 227.33 123.19) (end 224.79 123.19) (width 0.254) (layer B.Cu) (net 6))
@@
   (segment (start 170.18 120.65) (end 171.45 120.65) (width 0.254) (layer F.Cu) (net 6))
   (segment (start 171.45 120.65) (end 173.99 120.65) (width 0.254) (layer F.Cu) (net 6))
-  (segment (start 149.86 124.46) (end 149.86 121.92) (width 0.254) (layer F.Cu) (net 6))
   (segment (start 149.86 121.92) (end 149.86 116.84) (width 0.254) (layer F.Cu) (net 6))
   (segment (start 149.86 114.3) (end 149.86 116.84) (width 0.254) (layer F.Cu) (net 6))
@@
   (segment (start 193.04 125.73) (end 194.31 124.46) (width 0.254) (layer F.Cu) (net 15))
   (segment (start 181.61 125.73) (end 181.61 125.73) (width 0.254) (layer F.Cu) (net 15))
-  (segment (start 154.94 121.92) (end 186.69 121.92) (width 0.254) (layer B.Cu) (net 16))
+  (segment (start 158.75 121.92) (end 157.48 120.65) (width 0.254) (layer B.Cu) (net 16))
+  (segment (start 160.02 121.92) (end 158.75 121.92) (width 0.254) (layer B.Cu) (net 16))
+  (segment (start 153.67 123.19) (end 154.94 124.46) (width 0.254) (layer B.Cu) (net 16) (status 800000))
+  (segment (start 153.67 120.65) (end 153.67 123.19) (width 0.254) (layer B.Cu) (net 16))
+  (segment (start 157.48 120.65) (end 153.67 120.65) (width 0.254) (layer B.Cu) (net 16))
+  (segment (start 207.01 120.65) (end 205.74 119.38) (width 0.254) (layer F.Cu) (net 16))
+  (segment (start 203.2 119.38) (end 205.74 119.38) (width 0.254) (layer F.Cu) (net 16))
+  (via (at 203.2 119.38) (size 0.889) (layers F.Cu B.Cu) (net 16))
+  (segment (start 160.02 121.92) (end 160.02 121.92) (width 0.254) (layer B.Cu) (net 16))
+  (segment (start 160.02 121.92) (end 186.69 121.92) (width 0.254) (layer B.Cu) (net 16))
   (segment (start 187.96 120.65) (end 200.66 120.65) (width 0.254) (layer B.Cu) (net 16))
   (segment (start 186.69 121.92) (end 187.96 120.65) (width 0.254) (layer B.Cu) (net 16))
   (segment (start 200.66 119.38) (end 200.66 120.65) (width 0.254) (layer B.Cu) (net 16))
   (segment (start 200.66 119.38) (end 203.2 119.38) (width 0.254) (layer B.Cu) (net 16))
-  (via (at 203.2 119.38) (size 0.889) (layers F.Cu B.Cu) (net 16))
-  (segment (start 203.2 119.38) (end 205.74 119.38) (width 0.254) (layer F.Cu) (net 16))
-  (segment (start 207.01 120.65) (end 205.74 119.38) (width 0.254) (layer F.Cu) (net 16))
   (segment (start 194.31 114.3) (end 207.01 114.3) (width 0.254) (layer B.Cu) (net 17))
   (segment (start 154.94 114.3) (end 194.31 114.3) (width 0.254) (layer B.Cu) (net 17))
@@
   (segment (start 213.36 116.84) (end 210.82 116.84) (width 0.254) (layer F.Cu) (net 18))
   (segment (start 214.63 118.11) (end 213.36 116.84) (width 0.254) (layer F.Cu) (net 18))
-  (segment (start 154.94 124.46) (end 184.15 124.46) (width 0.254) (layer B.Cu) (net 19))
+  (segment (start 161.29 124.46) (end 157.48 124.46) (width 0.254) (layer B.Cu) (net 19))
+  (segment (start 157.48 124.46) (end 154.94 121.92) (width 0.254) (layer B.Cu) (net 19) (status 800000))
+  (segment (start 161.29 124.46) (end 161.29 124.46) (width 0.254) (layer B.Cu) (net 19))
+  (segment (start 161.29 124.46) (end 184.15 124.46) (width 0.254) (layer B.Cu) (net 19))
   (segment (start 200.66 123.19) (end 201.93 124.46) (width 0.254) (layer B.Cu) (net 19))
   (segment (start 185.42 123.19) (end 200.66 123.19) (width 0.254) (layer B.Cu) (net 19))
@@
   (segment (start 201.93 124.46) (end 201.93 124.46) (width 0.254) (layer B.Cu) (net 19))
   (segment (start 201.93 124.46) (end 217.17 124.46) (width 0.254) (layer B.Cu) (net 19))
+  (segment (start 217.17 124.46) (end 218.44 123.19) (width 0.254) (layer B.Cu) (net 19))
+  (via (at 218.44 123.19) (size 0.889) (layers F.Cu B.Cu) (net 19))
   (segment (start 217.17 121.92) (end 217.17 120.65) (width 0.254) (layer F.Cu) (net 19))
   (segment (start 218.44 123.19) (end 217.17 121.92) (width 0.254) (layer F.Cu) (net 19))
-  (via (at 218.44 123.19) (size 0.889) (layers F.Cu B.Cu) (net 19))
-  (segment (start 217.17 124.46) (end 218.44 123.19) (width 0.254) (layer B.Cu) (net 19))
   (segment (start 208.28 125.73) (end 209.55 127) (width 0.254) (layer F.Cu) (net 22))
   (segment (start 209.55 127) (end 219.71 127) (width 0.254) (layer F.Cu) (net 22))
