File: balance_jeanne/balance_jeanne.kicad_pcb (KiCad board)
At the start: 2 copper layers, 85.1 x 55.2 mm, 13 parts, among them P1 Digital, P10 rotary, P2 Analog, P3 CONN_1, P4 CONN_1, P5 CONN_1, P6 CONN_1, P7 bouton, P8 lcd_4x20, P9 balance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

Commit message: update balance jeanne
Aucune idée des modifs en cours... :-P
Parts:
- added P11: balance_serial, Pin_Headers:Pin_Header_Straight_1x04_Pitch2.54mm, F.Cu at (173.7, 101.9)
- U1: moved to B.Cu
- moved U1 5.26 mm to (175.1, 90.0), turned to 180 degrees
Connections:
- P9 pad 1: Net-(P9-Pad1) -> /IO0_3
- P9 pad 10: Net-(P9-Pad10) -> /IO1_0
- P9 pad 2: Net-(P9-Pad2) -> /IO0_2
- P9 pad 3: Net-(P9-Pad3) -> /IO0_4
- P9 pad 4: Net-(P9-Pad4) -> /IO0_1
- P9 pad 5: Net-(P9-Pad5) -> /IO0_5
- P9 pad 6: Net-(P9-Pad6) -> /IO0_0
- P9 pad 7: Net-(P9-Pad7) -> /IO0_6
- P9 pad 8: Net-(P9-Pad8) -> /IO1_1
- P9 pad 9: Net-(P9-Pad9) -> /IO0_7
- U1 pad 10: Net-(U1-Pad10) -> /IO0_6
- U1 pad 11: Net-(U1-Pad11) -> /IO0_7
- U1 pad 13: Net-(P9-Pad1) -> /IO1_0
- U1 pad 14: Net-(P9-Pad2) -> /IO1_1
- U1 pad 15: Net-(P9-Pad3) -> /IO1_2
- U1 pad 16: Net-(P9-Pad4) -> /IO1_3
- U1 pad 17: Net-(P9-Pad5) -> /IO1_4
- U1 pad 18: Net-(P9-Pad6) -> /IO1_5
- U1 pad 19: Net-(P9-Pad7) -> /IO1_6
- U1 pad 20: Net-(P9-Pad8) -> /IO1_7
- U1 pad 4: Net-(P9-Pad9) -> /IO0_0
- U1 pad 5: Net-(P9-Pad10) -> /IO0_1
- U1 pad 6: Net-(U1-Pad6) -> /IO0_2
- U1 pad 7: Net-(U1-Pad7) -> /IO0_3
- U1 pad 8: Net-(U1-Pad8) -> /IO0_4
- U1 pad 9: Net-(U1-Pad9) -> /IO0_5
Routing:
- net +5V: track 22.3 -> 87.9 mm, vias 2 -> 5
- net /IO0_0: track 0.00 -> 46.5 mm
- net /IO0_1: track 0.00 -> 41.6 mm
- net Net-(P9-Pad8): track 39.7 -> 0.00 mm
- net /IO1_1: track 0.00 -> 35.5 mm
- net Net-(P9-Pad6): track 33.6 -> 0.00 mm
- net Net-(P9-Pad10): track 28.4 -> 0.00 mm
- net Net-(P9-Pad4): track 27.6 -> 0.00 mm
- net Net-(P9-Pad9): track 25.1 -> 0.00 mm
- net GND: track 147.7 -> 172.7 mm, vias 2 -> 4
- net /IO1_0: track 0.00 -> 23.2 mm
- net Net-(P9-Pad7): track 22.8 -> 0.00 mm
- net /IO0_2: track 0.00 -> 22.6 mm
- net /A3: track 0.00 -> 20.9 mm
- net Net-(P9-Pad2): track 20.2 -> 0.00 mm
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- added copper zone on B.Cu, net GND
- removed copper zone on F.Cu, net GND
Other:
- board size 85.1 x 55.2 mm -> 88.9 x 55.6 mm
- net class Default: clearance 0.2 -> 0.25; trace_width 0.25 -> 0.5
- rule trace_clearance: 0.2 -> 0.25
